File: Design/H0FR8.brd (EAGLE design)
At the start: 34.6 x 30 mm, 24 parts, among them P1 HEXABIT_17.32_NO_P6, Q1 TLP184_GR-TPL,SE, U1 STM32G0B1CEU6N, U2 T2035H-6GD2PAK_T2550_STM-M, U3 VOT8121AM-VT, X1 XTALL_CSTCE8M00G52

Commit message: Stage1
Parts:
- added AC_MAINS, LOAD: (no value), HEXABITZ_CONNECTION_PARTS:1546111-2
- added C12, CSN2: 100nF, HEXABITZ_RCLS:C-0603
- added C13: 1nF, HEXABITZ_RCLS:C-0603
- added C9, CSN1: 10nF, HEXABITZ_RCLS:C-0603
- added D2: RED, Hexabitz:VLMS1300-GS08
- added R10, R5, RSN1: 100, HEXABITZ_RCLS:R-0603
- added R6: 390, HEXABITZ_RCLS:R-0603
- added R7: 180, HEXABITZ_RCLS:R-0603
- added R8: 3.3k, HEXABITZ_RCLS:R-0603
- added R9: 47, HEXABITZ_RCLS:R-0603
- added RSN2: 1.5k, HEXABITZ_RCLS:R-0603
- added RV1: MOVS4032V275, HEXABITZ_RCLS:MOVS4032V275
- added U4: TLP184_GR-TPL,SE, HEXABITZ_ICs:SOIC127P700X230-6N
- C5: value 100nF -> 1nF
- Q1: value TLP184_GR-TPL,SE -> MMBT3904LT1; device HEXABITZ_ICs:SOIC127P700X230-6N -> HEXABITZ_RCLS:MMBT3904LT1
- R4: value 0.0R -> 1k
- moved Q1 32.1 mm to (19.2, -8.41), flipped to the top, turned to 0 degrees
- moved C5 17.4 mm to (0.32, -9.21)
Connections:
- new net A2: LOAD.2, RSN1.2, RSN2.2, RV1.1, U2.2
- new net AC_MAINS_L: AC_MAINS.1, LOAD.1
- new net AC_MAINS_N: AC_MAINS.2, C9.2, CSN1.2, CSN2.2, R4.1, RV1.2, U2.1
- new net N$10: C12.1, R5.2, R9.2
- new net N$11: C12.2, Q1.3, R5.1
- new net N$12: R9.1, U3.2
- new net N$13: C5.1, Q1.1, R8.1
- new net N$4: CSN1.1, RSN1.1
- new net N$7: CSN2.1, R6.2, RSN2.1
- new net N$8: R6.1, U3.4
- new net N$9: D2.C, R7.2
- new net TRIAC_G: C9.1, R4.2, U2.3, U3.3
- new net ZC_DETECT: C13.1, R10.2, U4.6
- net GND: now also C13.2, Q1.2, U4.4
- net SSR: now also C5.2, R8.2
- net VDD: now also D2.A, R10.1, U3.1

Commit message: stage2
Parts:
- added D4: STMICROELECTRONICS_BAT46ZFILMSTMICROELECTRONICS_BAT46ZFILM_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, HEXABITZ_RCLS:STMICROELECTRONICS_BAT46ZFILM_3
- added R11: 100k, HEXABITZ_RCLS:R-0603
- D2: value RED -> BOURNS_CDSOD323-T03SCBOURNS_CDSOD323-T03SC_0_0; device Hexabitz:VLMS1300-GS08 -> HEXABITZ_RCLS:BOURNS_CDSOD323-T03SC_0
- D3: value BOURNS_CDSOD323-T03SCBOURNS_CDSOD323-T03SC_0_0 -> STMICROELECTRONICS_BAT46ZFILMSTMICROELECTRONICS_BAT46ZFILM_0_3; device HEXABITZ_RCLS:BOURNS_CDSOD323-T03SC_0 -> HEXABITZ_RCLS:STMICROELECTRONICS_BAT46ZFILM_3
- R10: value 100 -> 100k
- R7: value 180 -> 33k
- moved D3 38.6 mm to (0.95, -29.7), flipped to the top, turned to 0 degrees
- moved D2 36.3 mm to (-7.62, 7.94), flipped to the bottom, turned to 270 degrees
- moved R10 23.7 mm to (-4.92, -34.8)
- moved R7 14.3 mm to (8.57, -15.2)
- renumbered CSN1 to C10, CSN2 to C11, RSN1 to R12, RSN2 to R13
Connections:
- removed net N$9: D2.C, R7.2
- new net N$14: D3.2, D4.2
- new net N$15: D3.1, R11.1, U4.1
- new net N$16: D4.1, R10.1, U4.3
- net AC_MAINS_L: now also R11.2
- net AC_MAINS_N: now also R10.2
- net GND: now also D2.2; no longer D3.2
- net VDD: now also D2.1, R7.1; no longer D2.A, D3.1, R10.1
- net ZC_DETECT: now also R7.2; no longer R10.2

Commit message: Final schematic design
Parts:
- C11: value 100nF -> 47nF
- moved R9 49.5 mm to (-26.5, -45.6)
- moved R11 29.0 mm to (-26.5, -50.2)
- moved R10 5.58 mm to (-6.35, -29.4)
Connections:
- net N$3 renamed LED_INDICATOR
- removed net N$12: R9.1, U3.2
- removed net SSR: C5.2, R8.2, U1.43
- new net AGND: C3.2, C7.2, R3.2, U1.7
- new net N$3: R9.1, U3.1
- new net TRIAC_TRIGGER: C5.2, R8.2, U1.20
- net AC_MAINS_L: now also R10.2; no longer R11.2
- net AC_MAINS_N: now also R11.2; no longer R10.2
- net GND: now also R3.1; no longer R3.2
- net N$10: now also U3.2; no longer R9.2
- net N$15: now also R10.1; no longer R11.1
- net N$16: now also R11.1; no longer R10.1
- net VDD: now also FB1.1, R9.2; no longer FB1.2, U3.1
- net VDDA: now also FB1.2; no longer FB1.1
- net VSSA: no longer C3.2, C7.2, R3.1, U1.7
- net ZC_DETECT: now also U1.19
Routing:
- net VDD: track 6.79 -> 0.94 mm, vias 2 -> 0
- net LED_INDICATOR: track 2.14 -> 0.00 mm
- net SSR: track 1.23 -> 0.00 mm
- net VSSA: track 4.72 -> 3.74 mm
- net GND: track 10.8 -> 9.81 mm

Commit message: Schematic modification
Parts:
- added R14: 47, HEXABITZ_RCLS:R-0603
Connections:
- new net N$9: C5.2, R14.1
- net TRIAC_TRIGGER: now also R14.2; no longer C5.2
Changed lines of the file:
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@@
 <attribute name="TOLERANCE" value="" x="-6.985" y="-19.84375" size="1.778" layer="27" display="off"/>
 <attribute name="VALUE" x="-7.62" y="-21.74875" size="1.016" layer="27"/>
-<attribute name="VOLTAGE_RATING" value="" x="-6.985" y="-19.84375" size="1.778" layer="27" display="off"/>
+<attribute name="VOLTAGE_RATING" value="35V" x="-6.985" y="-19.84375" size="1.778" layer="27" display="off"/>
 </element>
 <element name="R6" library="HEXABITZ_RCLS" library_urn="urn:adsk.eagle:library:20064561" package="R-0603" package3d_urn="urn:adsk.eagle:package:1435818/6" value="390" x="-4.7625" y="-8.255" smashed="yes">
@@
 <attribute name="TOLERANCE" value="±5%" x="-26.51125" y="-50.165" size="1.778" layer="27" display="off"/>
 <attribute name="VALUE" x="-27.14625" y="-52.07" size="1.016" layer="27"/>
+</element>
+<element name="R14" library="HEXABITZ_RCLS" library_urn="urn:adsk.eagle:library:20064561" package="R-0603" package3d_urn="urn:adsk.eagle:package:1435818/6" value="47" x="-26.51125" y="-54.76875" smashed="yes">
+<attribute name="MFN" value="Yageo" x="-26.51125" y="-54.76875" size="1.778" layer="27" display="off"/>
+<attribute name="MPN" value="RC0402FR-07100RL" x="-26.51125" y="-54.76875" size="1.778" layer="27" display="off"/>
+<attribute name="NAME" x="-27.14625" y="-54.13375" size="1.016" layer="25"/>
+<attribute name="OCTOPART_URL" value="https://octopart.com/crcw0603110rfkea-vishay-39455532" x="-26.51125" y="-54.76875" size="1.778" layer="27" display="off"/>
+<attribute name="RESISTANCE" value="110.0 Ω" x="-26.51125" y="-54.76875" size="1.778" layer="27" display="off"/>
+<attribute name="TOLERANCE" value="±1%" x="-26.51125" y="-54.76875" size="1.778" layer="27" display="off"/>
+<attribute name="VALUE" x="-27.14625" y="-56.67375" size="1.016" layer="27"/>
 </element>
 </elements>
@@
 <signal name="TRIAC_TRIGGER">
 <contactref element="R8" pad="2"/>
-<contactref element="C5" pad="2"/>
 <contactref element="U1" pad="20"/>
-<wire x1="-0.59145" y1="4.5575" x2="1.1675" y2="-9.2075" width="0" layer="19" extent="1-16"/>
-<wire x1="18.63" y1="-18.89125" x2="1.1675" y2="-9.2075" width="0" layer="19" extent="1-1"/>
+<contactref element="R14" pad="2"/>
+<wire x1="18.63" y1="-18.89125" x2="-25.66125" y2="-54.76875" width="0" layer="19" extent="1-1"/>
+<wire x1="-0.59145" y1="4.5575" x2="18.63" y2="-18.89125" width="0" layer="19" extent="1-16"/>
 </signal>
 <signal name="LED_INDICATOR">
@@
 <wire x1="3.53875" y1="7.6874" x2="6.72375" y2="10.63625" width="0" layer="19" extent="16-16"/>
 </signal>
+<signal name="N$9">
+<contactref element="C5" pad="2"/>
+<contactref element="R14" pad="1"/>
+<wire x1="1.1675" y1="-9.2075" x2="-27.36125" y2="-54.76875" width="0" layer="19" extent="1-1"/>
+</signal>
 </signals>

Commit message: Schematic modification
Parts:
- C2, C3, C4: device HEXABITZ_RCLS:C-0805-POL -> HEXABITZ_RCLS:C-0603-POL
- moved R11 56.7 mm to (-24.1, 6.51)
- moved R14 56.7 mm to (-24.1, 1.91)
- moved R9 56.7 mm to (-24.1, 11.1)
- moved C4 29.8 mm to (23.5, 2.86), flipped to the top, turned to 0 degrees
- moved C2 18.4 mm to (23.5, 7.78), flipped to the top, turned to 0 degrees
- moved C3 17.6 mm to (23.5, 12.7), flipped to the top, turned to 0 degrees

Commit message: Schematic modification
Parts:
- added R15: 100k, HEXABITZ_RCLS:R-0603
Connections:
- net GND: now also R15.2
- net N$13: now also R15.1
Changed lines of the file:
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@@
 <attribute name="VOLTAGE_RATING" value="25V" x="23.495" y="2.8575" size="1.778" layer="27" display="off"/>
+</element>
+<element name="R15" library="HEXABITZ_RCLS" library_urn="urn:adsk.eagle:library:20064561" package="R-0603" package3d_urn="urn:adsk.eagle:package:1435818/6" value="100k" x="-26.51125" y="-43.02125" smashed="yes">
+<attribute name="MFN" value="Yageo" x="-26.51125" y="-43.02125" size="1.778" layer="27" display="off"/>
+<attribute name="MPN" value="RC0603JR-070RL" x="-26.51125" y="-43.02125" size="1.778" layer="27" display="off"/>
+<attribute name="NAME" x="-27.14625" y="-42.38625" size="1.016" layer="25"/>
+<attribute name="OCTOPART_URL" value="https://octopart.com/crcw06032k40jnea-vishay-40298967" x="-26.51125" y="-43.02125" size="1.778" layer="27" display="off"/>
+<attribute name="RESISTANCE" value="2400.0 Ω" x="-26.51125" y="-43.02125" size="1.778" layer="27" display="off"/>
+<attribute name="TOLERANCE" value="±5%" x="-26.51125" y="-43.02125" size="1.778" layer="27" display="off"/>
+<attribute name="VALUE" x="-27.14625" y="-44.92625" size="1.016" layer="27"/>
 </element>
 </elements>
@@
 <contactref element="U1" pad="30"/>
 <contactref element="C4" pad="2"/>
-<wire x1="1.1675" y1="-21.11375" x2="24.345" y2="2.8575" width="0" layer="19" extent="1-1"/>
+<contactref element="R15" pad="2"/>
+<wire x1="1.1675" y1="-21.11375" x2="-25.66125" y2="-43.02125" width="0" layer="19" extent="1-1"/>
 <wire x1="3.96875" y1="0.635" x2="1.1675" y2="-21.11375" width="0" layer="19" extent="1-1"/>
 <wire x1="3.96875" y1="1.905" x2="3.96875" y2="0.635" width="0" layer="19" extent="1-1"/>
@@
 <wire x1="-16.52" y1="14.9225" x2="-10.63625" y2="19.84375" width="0" layer="19" extent="16-16"/>
 <wire x1="8.26" y1="29.2325" x2="11.27125" y2="18.57375" width="0" layer="19" extent="16-16"/>
-<wire x1="20.15875" y1="-9.51375" x2="8.26" y2="0.6125" width="0" layer="19" extent="1-16"/>
+<wire x1="24.345" y1="2.8575" x2="10.63625" y2="4.445" width="0" layer="19" extent="1-1"/>
+<wire x1="20.15875" y1="-9.51375" x2="24.345" y2="2.8575" width="0" layer="19" extent="1-1"/>
 </signal>
 <signal name="VDD">
@@
 <contactref element="Q1" pad="1"/>
 <contactref element="C5" pad="1"/>
-<wire x1="18.25875" y1="-9.51375" x2="16.93" y2="-18.89125" width="0" layer="19" extent="1-1"/>
-<wire x1="-0.5325" y1="-9.2075" x2="18.25875" y2="-9.51375" width="0" layer="19" extent="1-1"/>
+<contactref element="R15" pad="1"/>
+<wire x1="-0.5325" y1="-9.2075" x2="-27.36125" y2="-43.02125" width="0" layer="19" extent="1-1"/>
+<wire x1="18.25875" y1="-9.51375" x2="-0.5325" y2="-9.2075" width="0" layer="19" extent="1-1"/>
+<wire x1="16.93" y1="-18.89125" x2="18.25875" y2="-9.51375" width="0" layer="19" extent="1-1"/>
 </signal>
 <signal name="N$10">

Commit message: Edit the description
Parts:
- moved AC_MAINS 64.4 mm to (-2.54, 25.7)
- moved LOAD 58.4 mm to (8.73, 25.7)
Changed lines of the file:
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@@
 <attribute name="VALUE" x="-20.79625" y="-15.24" size="1.27" layer="27" align="center"/>
 </element>
-<element name="LOAD" library="HEXABITZ_CONNECTION_PARTS" library_urn="urn:adsk.eagle:library:20064553" package="1546111-2" package3d_urn="urn:adsk.eagle:package:19666461/4" value="" x="-20.955" y="-24.60625" smashed="yes">
-<attribute name="MFN" value="TE Connectivity" x="-20.955" y="-24.60625" size="1.778" layer="27" display="off"/>
-<attribute name="MPN" value="1546111-2" x="-20.955" y="-24.60625" size="1.778" layer="27" display="off"/>
-<attribute name="NAME" x="-27.395" y="-31.39625" size="1.016" layer="25"/>
-<attribute name="OCTOPART_URL" value="https://octopart.com/1546111-2-te+connectivity-40393355" x="-20.955" y="-24.60625" size="1.778" layer="27" display="off"/>
-<attribute name="VALUE" x="-27.395" y="-32.80625" size="1.016" layer="27"/>
-</element>
-<element name="AC_MAINS" library="HEXABITZ_CONNECTION_PARTS" library_urn="urn:adsk.eagle:library:20064553" package="1546111-2" package3d_urn="urn:adsk.eagle:package:19666461/4" value="" x="-20.955" y="-36.03625" smashed="yes">
-<attribute name="MFN" value="TE Connectivity" x="-20.955" y="-36.03625" size="1.778" layer="27" display="off"/>
-<attribute name="MPN" value="1546111-2" x="-20.955" y="-36.03625" size="1.778" layer="27" display="off"/>
-<attribute name="NAME" x="-25.01375" y="13.8475" size="1.016" layer="25"/>
-<attribute name="OCTOPART_URL" value="https://octopart.com/1546111-2-te+connectivity-40393355" x="-20.955" y="-36.03625" size="1.778" layer="27" display="off"/>
-<attribute name="VALUE" x="-27.395" y="-44.23625" size="1.016" layer="27"/>
+<element name="LOAD" library="HEXABITZ_CONNECTION_PARTS" library_urn="urn:adsk.eagle:library:20064553" package="1546111-2" package3d_urn="urn:adsk.eagle:package:19666461/4" value="" x="8.73125" y="25.7175" smashed="yes">
+<attribute name="MFN" value="TE Connectivity" x="8.73125" y="25.7175" size="1.778" layer="27" display="off"/>
+<attribute name="MPN" value="1546111-2" x="8.73125" y="25.7175" size="1.778" layer="27" display="off"/>
+<attribute name="NAME" x="2.29125" y="18.9275" size="1.016" layer="25"/>
+<attribute name="OCTOPART_URL" value="https://octopart.com/1546111-2-te+connectivity-40393355" x="8.73125" y="25.7175" size="1.778" layer="27" display="off"/>
+<attribute name="VALUE" x="2.29125" y="17.5175" size="1.016" layer="27"/>
+</element>
+<element name="AC_MAINS" library="HEXABITZ_CONNECTION_PARTS" library_urn="urn:adsk.eagle:library:20064553" package="1546111-2" package3d_urn="urn:adsk.eagle:package:19666461/4" value="" x="-2.54" y="25.7175" smashed="yes">
+<attribute name="MFN" value="TE Connectivity" x="-2.54" y="25.7175" size="1.778" layer="27" display="off"/>
+<attribute name="MPN" value="1546111-2" x="-2.54" y="25.7175" size="1.778" layer="27" display="off"/>
+<attribute name="NAME" x="-6.59875" y="75.60125" size="1.016" layer="25"/>
+<attribute name="OCTOPART_URL" value="https://octopart.com/1546111-2-te+connectivity-40393355" x="-2.54" y="25.7175" size="1.778" layer="27" display="off"/>
+<attribute name="VALUE" x="-8.98" y="17.5175" size="1.016" layer="27"/>
 </element>
 <element name="R12" library="HEXABITZ_RCLS" library_urn="urn:adsk.eagle:library:20064561" package="R-0603" package3d_urn="urn:adsk.eagle:package:1435818/6" value="100" x="-6.985" y="-15.24" smashed="yes">
@@
 <contactref element="LOAD" pad="1"/>
 <contactref element="R10" pad="2"/>
-<wire x1="-23.495" y1="-36.03625" x2="-5.5" y2="-29.36875" width="0" layer="19" extent="1-1"/>
-<wire x1="-23.495" y1="-24.60625" x2="-23.495" y2="-36.03625" width="0" layer="19" extent="1-1"/>
+<wire x1="-5.08" y1="25.7175" x2="-5.5" y2="-29.36875" width="0" layer="19" extent="1-1"/>
+<wire x1="6.19125" y1="25.7175" x2="-5.08" y2="25.7175" width="0" layer="19" extent="1-1"/>
 </signal>
 <signal name="AC_MAINS_N">
@@
 <contactref element="C11" pad="2"/>
 <contactref element="R11" pad="2"/>
-<wire x1="-18.415" y1="-36.03625" x2="-23.28" y2="6.50875" width="0" layer="19" extent="1-1"/>
-<wire x1="-6.135" y1="-19.84375" x2="-18.415" y2="-36.03625" width="0" layer="19" extent="1-1"/>
+<wire x1="0" y1="25.7175" x2="-23.28" y2="6.50875" width="0" layer="19" extent="1-1"/>
+<wire x1="-6.135" y1="-19.84375" x2="0" y2="25.7175" width="0" layer="19" extent="1-1"/>
 <wire x1="1.32625" y1="-15.08125" x2="-6.135" y2="-19.84375" width="0" layer="19" extent="1-1"/>
 <wire x1="-16.59625" y1="-15.24" x2="-6.135" y2="-19.84375" width="0" layer="19" extent="1-1"/>
@@
 <contactref element="R13" pad="2"/>
 <wire x1="-6.135" y1="-15.24" x2="18.63" y2="-3.33375" width="0" layer="19" extent="1-1"/>
-<wire x1="-18.415" y1="-24.60625" x2="-6.135" y2="-15.24" width="0" layer="19" extent="1-1"/>
-<wire x1="-24.99625" y1="-15.24" x2="-18.415" y2="-24.60625" width="0" layer="19" extent="1-1"/>
+<wire x1="11.27125" y1="25.7175" x2="-6.135" y2="-15.24" width="0" layer="19" extent="1-1"/>
+<wire x1="-24.99625" y1="-15.24" x2="11.27125" y2="25.7175" width="0" layer="19" extent="1-1"/>
 <wire x1="0" y1="8.92175" x2="-24.99625" y2="-15.24" width="0" layer="19" extent="1-1"/>
 </signal>

Commit message: Intial Layout Design
Parts:
- removed AC_MAINS, LOAD: (no value), HEXABITZ_CONNECTION_PARTS:1546111-2
- removed C4: 4.7uF, HEXABITZ_RCLS:C-0603-POL
- removed C6: 100nF, HEXABITZ_RCLS:C-0603
- removed P1: HEXABIT_17.32_NO_P6, hexabitz_connectors:HEXABIT_17.32_NO_P6
- removed R15: 100k, HEXABITZ_RCLS:R-0603
- removed RV1: MOVS4032V275, HEXABITZ_RCLS:MOVS4032V275
- added U$1: HEXABIT_17.32_X3_NO_P1_P2_P3_P4_P5_P6_P11_P12, hexabitz_connectors:HEXABIT_17.32_X3_NO_P1_P2_P3_P4_P5_P6_P11_P12
- added U$2: FK244D2PAK, HEXABITZ_OTHER_PARTS:FK244D2PAK
- added U5: V275LA4P, HEXABITZ_RCLS:LA_07MM_LOW_LTF
- added X2: (no value), HEXABITZ_CONNECTION_PARTS:AK300/3
- C10, C11: device HEXABITZ_RCLS:C-0603 -> HEXABITZ_RCLS:C-0805
- R10, R11, R12, R13, R6: device HEXABITZ_RCLS:R-0603 -> HEXABITZ_RCLS:R-0805
- U1: value STM32G0B1CEU6N -> STM32G0B1CEU6QFN_B1CEU6_STM-L; device HEXABITZ_ICs:HEXABITZ_ICS_QFN_B1CEU6_STM-L -> HEXABITZ_ICs:QFN_B1CEU6_STM-L
- moved C12 76.6 mm to (2.54, 42.4), turned to 180 degrees
- moved D4 68.2 mm to (-5.24, 34.0), turned to 180 degrees
- moved D3 65.9 mm to (-9.05, 35.4), turned to 180 degrees
- moved C13 63.9 mm to (-5.40, 42.5)
- moved R5 63.6 mm to (2.54, 40.2)
- moved R7 60.9 mm to (-8.73, 43.2)
- moved R10 59.8 mm to (-9.84, 30.3), flipped to the bottom, turned to 270 degrees
- moved R8 59.4 mm to (-0.64, 37.6)
- moved Q1 52.8 mm to (-0.79, 40.5)
- moved C5 43.0 mm to (-0.32, 33.8)
- moved R9 41.8 mm to (5.87, 40.2), turned to 90 degrees
- moved R1 41.7 mm to (1.59, 45.1)
- moved R14 41.0 mm to (-0.64, 35.6)
- moved C2 40.6 mm to (-6.35, 35.2), flipped to the bottom
- moved D1 39.9 mm to (1.59, 45.1), turned to 270 degrees
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Connections:
- removed net AGND: C3.2, C7.2, R3.2, U1.7
- net A2: now also U$2.P$1, U$2.P$2, U5.2, X2.2; no longer LOAD.2, RV1.1
- net AC_MAINS_L: now also C10.2, C11.2, C9.2, R4.1, U2.1, U5.1, X2.3; no longer AC_MAINS.1, LOAD.1
- net AC_MAINS_N: now also X2.1; no longer AC_MAINS.2, C10.2, C11.2, C9.2, R4.1, RV1.2, U2.1
- net GND: now also U$1.PAD_PD12, U$1.PAD_PD17, U$1.PAD_PD19; no longer C4.2, C6.2, P1.PAD_PD10, P1.PAD_PD11, P1.PAD_PD12, P1.PAD_PD7, P1.PAD_PD8, P1.PAD_PD9, R15.2, U1.30
- net N$13: no longer R15.1
- net USART1_RX: now also U$1.PAD_PD8; no longer P1.PAD_PD4
- net USART1_TX: now also U$1.PAD_PU8; no longer P1.PAD_PU4
- net USART2_RX: now also U$1.PAD_PD1; no longer P1.PAD_PD2
- net USART2_TX: now also U$1.PAD_PU1; no longer P1.PAD_PU2
- net USART4_RX: now also U$1.PAD_PD3; no longer P1.PAD_PD1
- net USART4_TX: now also U$1.PAD_PU3; no longer P1.PAD_PU1
- net USART5_RX: no longer P1.PAD_PD5
- net USART5_TX: no longer P1.PAD_PU5
- net USART6_RX: now also U$1.PAD_PD2; no longer P1.PAD_PD3
- net USART6_TX: now also U$1.PAD_PU2; no longer P1.PAD_PU3
- net VDD: now also U$1.PAD_PU12, U$1.PAD_PU17, U$1.PAD_PU19; no longer C4.1, C6.1, P1.PAD_PU10, P1.PAD_PU11, P1.PAD_PU12, P1.PAD_PU7, P1.PAD_PU8, P1.PAD_PU9, U1.31
- net VSSA: now also C3.2, C7.2, R3.2, U1.7
Routing:
- net AC_MAINS_N: track 0.00 -> 37.1 mm
- net N$8: track 0.00 -> 33.9 mm, vias 0 -> 1
- net USART4_RX: track 25.9 -> 0.00 mm
- net USART4_TX: track 25.3 -> 0.00 mm, vias 1 -> 0
- net USART5_TX: track 21.3 -> 0.00 mm, vias 1 -> 0
- net USART5_RX: track 16.0 -> 0.00 mm
- net N$2: track 15.9 -> 0.00 mm, vias 1 -> 0
- net USART2_RX: track 14.2 -> 0.00 mm
- net USART2_TX: track 12.8 -> 0.00 mm, vias 1 -> 0
- net USART1_TX: track 12.1 -> 0.00 mm, vias 1 -> 0
- net CLK: track 11.2 -> 0.00 mm
- net USART1_RX: track 10.9 -> 0.00 mm
- net GND: track 9.81 -> 0.00 mm, vias 23 -> 0
- net USART6_TX: track 8.08 -> 0.00 mm, vias 1 -> 0
- net DATA: track 7.78 -> 0.00 mm
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- added copper zone on layer 1, net A2
- added copper zone on layer 16, net A2
- added copper zone on layer 1, net AC_MAINS_L
Other:
- board size 34.6 x 30 mm -> 60 x 60.6 mm
- board text added: "220V/10A (RMS)"
- board text added: "IN"
- board text added: "N"
- board text added: "OUT"
- board text removed: "600VAC/1.2A"
- board text removed: "P5"
