File: Design/H0FR8.brd (EAGLE design)
At the start: 60 x 60.6 mm, 43 parts, among them Q1 MMBT3904LT1, U1 STM32G0B1CEU6QFN_B1CEU6_STM-L, U2 T2035H-6GD2PAK_T2550_STM-M, U3 VOT8121AM-VT, U4 TLP184_GR-TPL,SE, U5 V275LA4P, X1 XTALL_CSTCE8M00G52

Commit message: - Fixed component's footprints and 3d packages.
Parts:
- U4: device HEXABITZ_ICs:SOIC127P700X230-6N -> HEXABITZ_ICs:SOIC254P700X230-4N
- moved TRIMBLE-LOGO2 2764.5 mm to (2000.0, 1959.1)
- moved R11 150.1 mm to (-0.95, -119.7), flipped to the top, turned to 180 degrees
- moved R10 137.6 mm to (-0.95, -107.0), flipped to the top, turned to 180 degrees
- moved R13 103.5 mm to (-0.95, -94.3), flipped to the top, turned to 180 degrees
- moved U4 94.3 mm to (-3.25, -54.9), turned to 0 degrees
- moved R6 89.2 mm to (-0.95, -81.6), flipped to the top
- moved R12 78.1 mm to (-0.95, -68.9), flipped to the top, turned to 180 degrees
- moved SWD 78.0 mm to (-2.54, -40.9), turned to 0 degrees
- moved C2 63.7 mm to (-0.85, -28.2), flipped to the top
- moved C3 52.0 mm to (-0.85, -15.5), flipped to the top
Routing:
- net N$8: track 33.9 -> 28.3 mm, vias 1 -> 2

Commit message: - Intial PCB design.
Parts:
- moved TRIMBLE-LOGO2 2785.0 mm to (20.5, -0.07)
- moved R11 149.6 mm to (-10.0, 29.7), turned to 270 degrees
- moved R10 114.5 mm to (-11.9, 6.99), turned to 270 degrees
- moved R13 110.1 mm to (-15.9, 14.8)
- moved R6 96.1 mm to (-12.6, 13.8), turned to 90 degrees
- moved U4 93.4 mm to (-6.74, 38.4)
- moved R12 82.6 mm to (-15.9, 12.4)
- moved SWD 78.7 mm to (9.82, 36.8), turned to 90 degrees
- moved C2 64.7 mm to (-6.45, 36.2), flipped to the bottom
- moved C3 51.1 mm to (-6.45, 35.3), flipped to the bottom
- moved R2 5.91 mm to (6.67, 36.0)
- moved R9 2.27 mm to (6.35, 42.4)
- moved X1 2.16 mm to (-7.30, 41.1)
- moved R1 1.94 mm to (3.17, 44.0)
- moved R 1.91 mm to (-3.33, 44.9)
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Routing:
- net GND: track 0.00 -> 92.6 mm, vias 0 -> 10
- net N$15: track 0.00 -> 53.3 mm, vias 0 -> 2
- net TRIAC_G: track 0.00 -> 46.1 mm
- net AC_MAINS_L: track 0.00 -> 27.6 mm, vias 0 -> 1
- net N$7: track 0.00 -> 20.5 mm, vias 0 -> 1
- net USART1_RX: track 0.00 -> 17.7 mm
- net USART1_TX: track 0.00 -> 16.9 mm, vias 0 -> 1
- net VDD: track 0.00 -> 15.9 mm, vias 0 -> 1
- net N$16: track 0.00 -> 14.9 mm
- net N$4: track 0.00 -> 14.5 mm, vias 0 -> 1
- net USART4_RX: track 0.00 -> 14.3 mm, vias 0 -> 2
- net ZC_DETECT: track 0.00 -> 13.9 mm, vias 0 -> 1
- net USART4_TX: track 0.00 -> 13.3 mm, vias 0 -> 1
- net USART6_TX: track 0.00 -> 12.0 mm, vias 0 -> 1
- net USART6_RX: track 0.00 -> 11.8 mm
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- added copper zone on layer 16, net GND
- added copper zone on layer 1, net VDD
