File: Design/H0FR8.sch (EAGLE design)
At the start: 24 parts, among them P1 HEXABIT_17.32_NO_P6, Q1 TLP184_GR-TPL,SE, U1 STM32G0B1CEU6N, U2 T2035H-6GD2PAK_T2550_STM-M, U3 VOT8121AM-VT, X1 XTALL_CSTCE8M00G52

Commit message: Stage1
Parts:
- added AC_MAINS, LOAD: (no value), HEXABITZ_CONNECTION_PARTS:1546111-2
- added C12, CSN2: 100nF, HEXABITZ_RCLS:C-0603
- added C13: 1nF, HEXABITZ_RCLS:C-0603
- added C9, CSN1: 10nF, HEXABITZ_RCLS:C-0603
- added D2: RED, Hexabitz:VLMS1300-GS08
- added R10, R5, RSN1: 100, HEXABITZ_RCLS:R-0603
- added R6: 390, HEXABITZ_RCLS:R-0603
- added R7: 180, HEXABITZ_RCLS:R-0603
- added R8: 3.3k, HEXABITZ_RCLS:R-0603
- added R9: 47, HEXABITZ_RCLS:R-0603
- added RSN2: 1.5k, HEXABITZ_RCLS:R-0603
- added RV1: MOVS4032V275, HEXABITZ_RCLS:MOVS4032V275
- added U4: TLP184_GR-TPL,SE, HEXABITZ_ICs:TLP184_GR-TPL,SE
- C5: value 100nF -> 1nF
- Q1: value TLP184_GR-TPL,SE -> MMBT3904LT1; device HEXABITZ_ICs:TLP184_GR-TPL,SE -> HEXABITZ_RCLS:MMBT3904LT1; MFN (none) -> ON Semiconductor; MPN (none) -> MMBT3904LT1G; OCTOPART_ID (none) -> 0bb6c2bc2200d471; OCTOPART_URL (none) -> http://octopart.com/mmbt3904lt1g-on+semiconductor-3280; POLARITY (none) -> NPN; POWER_DISSIPATION (none) -> 0.225 W; VOLTAGE_RATING_DC (none) -> 40.0 V
- R4: value 0.0R -> 1k
Connections:
- new net A2: LOAD.2, RSN1.2, RSN2.2, RV1.1, U2.A2
- new net AC_MAINS_L: AC_MAINS.1, LOAD.1
- new net AC_MAINS_N: AC_MAINS.2, C9.2, CSN1.2, CSN2.2, R4.1, RV1.2, U2.A1
- new net N$10: C12.1, R5.2, R9.2
- new net N$11: C12.2, Q1.C, R5.1
- new net N$12: R9.1, U3.C
- new net N$13: C5.1, Q1.B, R8.1
- new net N$4: CSN1.1, RSN1.1
- new net N$7: CSN2.1, R6.2, RSN2.1
- new net N$8: R6.1, U3.MT2
- new net N$9: D2.C, R7.2
- new net TRIAC_G: C9.1, R4.2, U2.G, U3.MT1
- new net ZC_DETECT: C13.1, R10.2, U4.COLLECTOR
- net GND: now also C13.2, Q1.E, U4.EMITTER
- net SSR: now also C5.2, R8.2
- net VDD: now also D2.A, R10.1, U3.A
Other:
- note added: "AC Dimmer Module"
- note removed: "Triac Dimmer Switch"
- moved on the sheet: C5, R4, U2, U3

Commit message: stage2
Parts:
- removed RSN2: 1.5k, HEXABITZ_RCLS:R-0603
- added D4: STMICROELECTRONICS_BAT46ZFILMSTMICROELECTRONICS_BAT46ZFILM_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, HEXABITZ_RCLS:STMICROELECTRONICS_BAT46ZFILMSTMICROELECTRONICS_BAT46ZFILM_0_3
- added R11: 100k, HEXABITZ_RCLS:R-0603
- added R13: 1.5k, HEXABITZ_RCLS:R-0603
- D2: value RED -> BOURNS_CDSOD323-T03SCBOURNS_CDSOD323-T03SC_0_0; device Hexabitz:VLMS1300-GS08 -> HEXABITZ_RCLS:BOURNS_CDSOD323-T03SCBOURNS_CDSOD323-T03SC_0_0; MFN Vishay -> (none); MPN VLMY1300-GS08 -> (none); OCTOPART_URL https://octopart.com/vlmy1300-gs08-vishay-21709204 -> (none)
- D3: value BOURNS_CDSOD323-T03SCBOURNS_CDSOD323-T03SC_0_0 -> STMICROELECTRONICS_BAT46ZFILMSTMICROELECTRONICS_BAT46ZFILM_0_3; device HEXABITZ_RCLS:BOURNS_CDSOD323-T03SCBOURNS_CDSOD323-T03SC_0_0 -> HEXABITZ_RCLS:STMICROELECTRONICS_BAT46ZFILMSTMICROELECTRONICS_BAT46ZFILM_0_3
- R10: value 100 -> 100k; MPN RC0402FR-07100RL -> RC0603JR-070RL; OCTOPART_URL https://octopart.com/crcw0603110rfkea-vishay-39455532 -> https://octopart.com/crcw06032k40jnea-vishay-40298967; RESISTANCE 110.0 Ω -> 2400.0 Ω; TOLERANCE ±1% -> ±5%
- R7: value 180 -> 33k; OCTOPART_URL https://octopart.com/erj-3geyj181v-panasonic-55403673 -> https://octopart.com/crcw0603110rfkea-vishay-39455532; RESISTANCE 180.0 Ω -> 110.0 Ω; TOLERANCE ±5% -> ±1%
- renumbered CSN1 to C10, CSN2 to C11, RSN1 to R12
Connections:
- removed net N$9: D2.C, R7.2
- new net N$14: D3.ANODE, D4.ANODE
- new net N$15: D3.CATHODE, R11.1, U4.ANODE_CATHODE
- new net N$16: D4.CATHODE, R10.1, U4.CATHODE_ANODE
- net A2: now also R13.2; no longer RSN2.2
- net AC_MAINS_L: now also R11.2
- net AC_MAINS_N: now also R10.2
- net GND: now also D2.C; no longer D3.C
- net N$7: now also R13.1; no longer RSN2.1
- net VDD: now also R7.1; no longer D3.A, R10.1
- net ZC_DETECT: now also R7.2; no longer R10.2
Other:
- note added: "MMSZ5225BT1G"
- moved on the sheet: C13, R10, R7, U4

Commit message: Final schematic design
Parts:
- C10: VOLTAGE_RATING (none) -> 400V
- C11: value 100nF -> 47nF; VOLTAGE_RATING (none) -> 400V
- R10, R11: POWER (none) -> 0.25W
- R12, R13, R6: POWER (none) -> 0.5W
Connections:
- net N$3 renamed LED_INDICATOR
- removed net N$12: R9.1, U3.C
- removed net SSR: C5.2, R8.2, U1.PB4
- new net AGND: C3.-, C7.2, R3.2, U1.VSS/VSSA
- new net N$3: R9.1, U3.A
- new net TRIAC_TRIGGER: C5.2, R8.2, U1.PB1
- net AC_MAINS_L: now also R10.2; no longer R11.2
- net AC_MAINS_N: now also R11.2; no longer R10.2
- net GND: now also R3.1; no longer R3.2
- net N$10: now also U3.C; no longer R9.2
- net N$15: now also R10.1; no longer R11.1
- net N$16: now also R11.1; no longer R10.1
- net VDD: now also FB1.1, R9.2; no longer FB1.2, U3.A
- net VDDA: now also FB1.2; no longer FB1.1
- net VSSA: no longer C3.-, C7.2, R3.1, U1.VSS/VSSA
- net ZC_DETECT: now also U1.PB0
Other:
- moved on the sheet: AC_MAINS, C1, C10, C11, C12, C13, C2, C3, C4, C5, C9, D1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

Commit message: Schematic modification
Parts:
- added R14: 47, HEXABITZ_RCLS:R-0603
- C9: VOLTAGE_RATING (none) -> 35V
Connections:
- new net N$9: C5.2, R14.1
- net TRIAC_TRIGGER: now also R14.2; no longer C5.2
Other:
- moved on the sheet: C12, C13, C5, C9, D3, D4, Q1, R10, R11, R5, R7, R8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

Commit message: Schematic modification
Parts:
- C2: device HEXABITZ_RCLS:C-0805-POL -> HEXABITZ_RCLS:C-0603-POL; CAPACITANCE (none) -> 1.00uF; MFN (none) -> Yageo; MPN (none) -> CC0805KKX7R7BB105; OCTOPART_URL (none) -> https://octopart.com/cc0805kkx7r7bb105-yageo-8376555?r=sp&s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; TOLERANCE (none) -> 10%; VOLTAGE_RATING (none) -> 16V
- C3, C4: device HEXABITZ_RCLS:C-0805-POL -> HEXABITZ_RCLS:C-0603-POL; CAPACITANCE (none) -> 4.7uF; MFN (none) -> Murata; MPN (none) -> GRM21BC81E475KA12L; OCTOPART_URL (none) -> https://octopart.com/grm21bc81e475ka12l-murata-10331911?r=s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; TOLERANCE (none) -> 10%; VOLTAGE_RATING (none) -> 25V
Connections:
- net AGND: now also C3.2; no longer C3.-
- net GND: now also C4.2; no longer C4.-
- net VDD: now also C4.1; no longer C4.+
- net VDDA: now also C2.1, C3.1; no longer C2.+, C3.+
- net VSSA: now also C2.2; no longer C2.-
Other:
- note added: "VDDA Coupling"
- note removed: "VDD\VDDA Coupling"
- moved on the sheet: C2, C3, C4

Commit message: Schematic modification
Parts:
- added R15: 100k, HEXABITZ_RCLS:R-0603
Connections:
- net GND: now also R15.2
- net N$13: now also R15.1
Changed lines of the file:
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@@
 <attribute name="VOLTAGE_RATING" value="25V"/>
 </part>
+<part name="R15" library="HEXABITZ_RCLS" library_urn="urn:adsk.eagle:library:20064561" deviceset="R-0603" device="" package3d_urn="urn:adsk.eagle:package:1435818/6" value="100k">
+<attribute name="MFN" value="Yageo"/>
+<attribute name="MPN" value="RC0603JR-070RL"/>
+<attribute name="OCTOPART_URL" value="https://octopart.com/crcw06032k40jnea-vishay-40298967"/>
+<attribute name="RESISTANCE" value="2400.0 Ω"/>
+<attribute name="TOLERANCE" value="±5%"/>
+</part>
+<part name="GND13" library="supply1" library_urn="urn:adsk.eagle:library:371" deviceset="GND" device=""/>
 </parts>
 <sheets>
@@
 <attribute name="VALUE" x="62.23" y="112.522" size="1.778" layer="96" rot="R180"/>
 </instance>
-<instance part="GND4" gate="1" x="77.47" y="102.87" smashed="yes">
-<attribute name="VALUE" x="74.93" y="100.33" size="1.778" layer="96"/>
+<instance part="GND4" gate="1" x="77.47" y="97.79" smashed="yes">
+<attribute name="VALUE" x="74.93" y="95.25" size="1.778" layer="96"/>
 </instance>
 <instance part="C12" gate="G$1" x="71.755" y="129.54" smashed="yes">
@@
 <attribute name="VALUE" x="52.705" y="117.348" size="1.778" layer="96"/>
 </instance>
+<instance part="R15" gate="G$1" x="68.58" y="106.045" smashed="yes" rot="R270">
+<attribute name="NAME" x="70.485" y="106.2736" size="1.778" layer="95"/>
+<attribute name="VALUE" x="70.485" y="104.013" size="1.778" layer="96"/>
+</instance>
+<instance part="GND13" gate="1" x="68.58" y="97.79" smashed="yes">
+<attribute name="VALUE" x="66.04" y="95.25" size="1.778" layer="96"/>
+</instance>
 </instances>
 <busses>
@@
 <wire x1="68.58" y1="120.65" x2="68.58" y2="114.3" width="0.1524" layer="91"/>
 <junction x="68.58" y="114.3"/>
+<pinref part="R15" gate="G$1" pin="1"/>
+<wire x1="68.58" y1="111.125" x2="68.58" y2="114.3" width="0.1524" layer="91"/>
 </segment>
 </net>
@@
 <pinref part="Q1" gate="G$1" pin="E"/>
 <pinref part="GND4" gate="1" pin="GND"/>
-<wire x1="77.47" y1="109.22" x2="77.47" y2="105.41" width="0.1524" layer="91"/>
+<wire x1="77.47" y1="109.22" x2="77.47" y2="100.33" width="0.1524" layer="91"/>
 </segment>
 <segment>
@@
 <wire x1="163.195" y1="57.15" x2="163.195" y2="59.69" width="0.1524" layer="91"/>
 </segment>
+<segment>
+<pinref part="GND13" gate="1" pin="GND"/>
+<pinref part="R15" gate="G$1" pin="2"/>
+<wire x1="68.58" y1="100.965" x2="68.58" y2="100.33" width="0.1524" layer="91"/>
+</segment>
 </net>

Commit message: Edit the description
Other:
- note added: "10A RMS AC Dimmer"
- note removed: "AC Dimmer Module"
Changed lines of the file:
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@@
 <wire x1="231.14" y1="18.288" x2="231.14" y2="22.86" width="0.1524" layer="205"/>
 <text x="242.6462" y="6.1722" size="1.9304" layer="100" font="vector">www.hexabitz.com</text>
-<text x="182.4228" y="11.2014" size="1.9304" layer="101" font="vector">AC Dimmer Module</text>
+<text x="182.4228" y="11.2014" size="1.9304" layer="101" font="vector">10A RMS AC Dimmer</text>
 <text x="38.735" y="191.135" size="1.778" layer="150">VDD=3.3 Volts</text>
 <text x="168.825" y="94.82" size="1.778" layer="95">Vref Coupling</text>
@@
 <text x="199.4662" y="19.6342" size="1.9304" layer="100" font="vector">Title</text>
 <text x="180.9242" y="19.6342" size="1.9304" layer="102" font="vector">H0FR8</text>
-<text x="179.2478" y="11.2014" size="1.9304" layer="101" font="vector">AC Dimmer Module</text>
+<text x="179.2478" y="11.2014" size="1.9304" layer="101" font="vector">10A RMS AC Dimmer</text>
 <text x="206.3242" y="19.6342" size="1.9304" layer="101" font="vector">H0FR8_Frontend</text>
 <wire x1="168.91" y1="3.81" x2="168.91" y2="8.128" width="0.1524" layer="205"/>

Commit message: Intial Layout Design
Parts:
- removed AC_MAINS, LOAD: (no value), HEXABITZ_CONNECTION_PARTS:1546111-2
- removed C4: 4.7uF, HEXABITZ_RCLS:C-0603-POL
- removed C6: 100nF, HEXABITZ_RCLS:C-0603
- removed P1: HEXABIT_17.32_NO_P6, hexabitz_connectors:HEXABIT_17.32_NO_P6
- removed R15: 100k, HEXABITZ_RCLS:R-0603
- removed RV1: MOVS4032V275, HEXABITZ_RCLS:MOVS4032V275
- added U$1: HEXABIT_17.32_X3_NO_P1_P2_P3_P4_P5_P6_P11_P12, hexabitz_connectors:HEXABIT_17.32_X3_NO_P1_P2_P3_P4_P5_P6_P11_P12
- added U$2: FK244D2PAK, HEXABITZ_OTHER_PARTS:FK244D2PAK
- added U5: V275LA4P, HEXABITZ_RCLS:V275LA4P
- added X2: (no value), HEXABITZ_CONNECTION_PARTS:AK300/3
- C10: device HEXABITZ_RCLS:C-0603 -> HEXABITZ_RCLS:C-0805; MPN (none) -> C2012X7T2W103M085AA
- C11: device HEXABITZ_RCLS:C-0603 -> HEXABITZ_RCLS:C-0805; MPN (none) -> C2012X7T2W473K125AA
- R10: device HEXABITZ_RCLS:R-0603 -> HEXABITZ_RCLS:R-0805
- R11: device HEXABITZ_RCLS:R-0603 -> HEXABITZ_RCLS:R-0805; MFN Yageo -> (none); MPN RC0603JR-070RL -> ERJ-P06J104V; OCTOPART_URL https://octopart.com/crcw06032k40jnea-vishay-40298967 -> (none); POWER 0.25W -> (none); RESISTANCE 2400.0 Ω -> (none); TOLERANCE ±5% -> (none)
- R12: device HEXABITZ_RCLS:R-0603 -> HEXABITZ_RCLS:R-0805; MPN (none) -> ERJ-P06J101V
- R13: device HEXABITZ_RCLS:R-0603 -> HEXABITZ_RCLS:R-0805; MPN (none) -> ERJ-P06J152V
- R6: device HEXABITZ_RCLS:R-0603 -> HEXABITZ_RCLS:R-0805; MPN (none) -> ERJ-P06J391V
- U1: value STM32G0B1CEU6N -> STM32G0B1CEU6QFN_B1CEU6_STM-L; device HEXABITZ_ICs:STM32G0B1CEU6N -> HEXABITZ_ICs:STM32G0B1CEU6QFN_B1CEU6_STM-L
Connections:
- removed net AGND: C3.2, C7.2, R3.2, U1.VSS/VSSA
- net A2: now also U$2.H_S, U5.2, X2-2.KL; no longer LOAD.2, RV1.1
- net AC_MAINS_L: now also C10.2, C11.2, C9.2, R4.1, U2.A1, U5.1, X2-3.KL; no longer AC_MAINS.1, LOAD.1
- net AC_MAINS_N: now also X2-1.KL; no longer AC_MAINS.2, C10.2, C11.2, C9.2, R4.1, RV1.2, U2.A1
- net GND: now also U$1.GND1, U$1.GND2, U$1.GND3; no longer C4.2, C6.2, P1.GND1, P1.GND2, P1.GND3, P1.GND4, P1.GND5, P1.GND6, R15.2, U1.EPAD
- net N$13: no longer R15.1
- net USART1_RX: now also U$1.SD4; no longer P1.SD4
- net USART1_TX: now also U$1.SU4; no longer P1.SU4
- net USART2_RX: now also U$1.SD2; no longer P1.SD2
- net USART2_TX: now also U$1.SU2; no longer P1.SU2
- net USART4_RX: now also U$1.SD1; no longer P1.SD1
- net USART4_TX: now also U$1.SU1; no longer P1.SU1
- net USART5_RX: no longer P1.SD5
- net USART5_TX: no longer P1.SU5
- net USART6_RX: now also U$1.SD3; no longer P1.SD3
- net USART6_TX: now also U$1.SU3; no longer P1.SU3
- net VDD: now also U$1.VDD1, U$1.VDD2, U$1.VDD3; no longer C4.1, C6.1, P1.VDD1, P1.VDD2, P1.VDD3, P1.VDD4, P1.VDD5, P1.VDD6, U1.VDDIO2
- net VSSA: now also C3.2, C7.2, R3.2, U1.VSS/VSSA
Other:
- note added: "AC Dimmer Module"
- note removed: "10A RMS AC Dimmer"
- note removed: "VDDIO2 Coupling"
- moved on the sheet: D2
